File: PowerSupply_1_1.sch (KiCad schematic (older format))
At the start: 31 parts, among them Q4 IRF8721, U1 AP1117E33, U2 ADP2381, U3 TPS54428

Commit message: Added load resistor. Changed part references in consequence.
Parts:
- BT1: value ML2016 -> 3V LiMnO2; Part Number ML 2016 T6 -> ML2016 T6
- renumbered R10 to R11, R11 to R12, R12 to R13, R13 to R14, R14 to R15, R15 to R16, R16 to R17, R17 to R18
Changed lines of the file:
@@
 $EndComp
 $Comp
-L GND #PWR033
+L GND #PWR034
 U 1 1 528DE4FA
 P 4650 2950
-F 0 "#PWR033" H 4650 2950 30  0001 C CNN
+F 0 "#PWR034" H 4650 2950 30  0001 C CNN
 F 1 "GND" H 4650 2880 30  0001 C CNN
 F 2 "" H 4650 2950 60  0000 C CNN
@@
 $EndComp
 $Comp
-L GND #PWR034
+L GND #PWR035
 U 1 1 528DE509
 P 4950 2950
-F 0 "#PWR034" H 4950 2950 30  0001 C CNN
+F 0 "#PWR035" H 4950 2950 30  0001 C CNN
 F 1 "GND" H 4950 2880 30  0001 C CNN
 F 2 "" H 4950 2950 60  0000 C CNN
@@
 $EndComp
 $Comp
-L R R13
+L R R14
 U 1 1 528DE51A
 P 4350 2700
-F 0 "R13" V 4430 2700 40  0000 C CNN
+F 0 "R14" V 4430 2700 40  0000 C CNN
 F 1 "22k" V 4357 2701 40  0000 C CNN
 F 2 "Resistors_SMD:R_0805" V 4280 2700 30  0001 C CNN
@@
 $EndComp
 $Comp
-L R R14
+L R R15
 U 1 1 528DE53A
 P 4350 3600
-F 0 "R14" V 4430 3600 40  0000 C CNN
+F 0 "R15" V 4430 3600 40  0000 C CNN
 F 1 "3k" V 4357 3601 40  0000 C CNN
 F 2 "Resistors_SMD:R_0805" V 4280 3600 30  0001 C CNN
@@
 $EndComp
 $Comp
-L GND #PWR035
+L GND #PWR036
 U 1 1 528DE577
 P 4350 3950
-F 0 "#PWR035" H 4350 3950 30  0001 C CNN
+F 0 "#PWR036" H 4350 3950 30  0001 C CNN
 F 1 "GND" H 4350 3880 30  0001 C CNN
 F 2 "" H 4350 3950 60  0000 C CNN
@@
 $EndComp
 $Comp
-L GND #PWR036
+L GND #PWR037
 U 1 1 528DF20F
 P 3250 3850
-F 0 "#PWR036" H 3250 3850 30  0001 C CNN
+F 0 "#PWR037" H 3250 3850 30  0001 C CNN
 F 1 "GND" H 3250 3780 30  0001 C CNN
 F 2 "" H 3250 3850 60  0000 C CNN
@@
 $EndComp
 $Comp
-L GND #PWR037
+L GND #PWR038
 U 1 1 528DF2BC
 P 3550 3350
-F 0 "#PWR037" H 3550 3350 30  0001 C CNN
+F 0 "#PWR038" H 3550 3350 30  0001 C CNN
 F 1 "GND" H 3550 3280 30  0001 C CNN
 F 2 "" H 3550 3350 60  0000 C CNN
@@
 $EndComp
 $Comp
-L GND #PWR038
+L GND #PWR039
 U 1 1 528DF34E
 P 2400 3750
-F 0 "#PWR038" H 2400 3750 30  0001 C CNN
+F 0 "#PWR039" H 2400 3750 30  0001 C CNN
 F 1 "GND" H 2400 3680 30  0001 C CNN
 F 2 "" H 2400 3750 60  0000 C CNN
@@
 $EndComp
 $Comp
-L R R12
+L R R13
 U 1 1 528DF37F
 P 2800 4100
-F 0 "R12" V 2880 4100 40  0000 C CNN
+F 0 "R13" V 2880 4100 40  0000 C CNN
 F 1 "82k" V 2807 4101 40  0000 C CNN
 F 2 "Resistors_SMD:R_0805" V 2730 4100 30  0001 C CNN
@@
 $EndComp
 $Comp
-L R R10
+L R R11
 U 1 1 528E0FC8
 P 1300 2800
-F 0 "R10" V 1380 2800 40  0000 C CNN
+F 0 "R11" V 1380 2800 40  0000 C CNN
 F 1 "82k" V 1307 2801 40  0000 C CNN
 F 2 "Resistors_SMD:R_0805" V 1230 2800 30  0001 C CNN
@@
 $EndComp
 $Comp
-L GND #PWR039
+L GND #PWR040
 U 1 1 528E1066
 P 950 3050
-F 0 "#PWR039" H 950 3050 30  0001 C CNN
+F 0 "#PWR040" H 950 3050 30  0001 C CNN
 F 1 "GND" H 950 2980 30  0001 C CNN
 F 2 "" H 950 3050 60  0000 C CNN
@@
 $EndComp
 $Comp
-L R R15
+L R R16
 U 1 1 528E1D22
 P 6450 2350
-F 0 "R15" V 6530 2350 40  0000 C CNN
+F 0 "R16" V 6530 2350 40  0000 C CNN
 F 1 "10k" V 6457 2351 40  0000 C CNN
 F 2 "Resistors_SMD:R_0805" V 6380 2350 30  0001 C CNN
@@
 $EndComp
 $Comp
-L GND #PWR040
+L GND #PWR041
 U 1 1 528E209F
 P 6100 3300
-F 0 "#PWR040" H 6100 3300 30  0001 C CNN
+F 0 "#PWR041" H 6100 3300 30  0001 C CNN
 F 1 "GND" H 6100 3230 30  0001 C CNN
 F 2 "" H 6100 3300 60  0000 C CNN
@@
 $EndComp
 $Comp
-L GND #PWR041
+L GND #PWR042
 U 1 1 528E20AE
 P 6800 3500
-F 0 "#PWR041" H 6800 3500 30  0001 C CNN
+F 0 "#PWR042" H 6800 3500 30  0001 C CNN
 F 1 "GND" H 6800 3430 30  0001 C CNN
 F 2 "" H 6800 3500 60  0000 C CNN
@@
 $EndComp
 $Comp
-L R R17
+L R R18
 U 1 1 528E22B3
 P 9950 2700
-F 0 "R17" V 10030 2700 40  0000 C CNN
+F 0 "R18" V 10030 2700 40  0000 C CNN
 F 1 "33k" V 9957 2701 40  0000 C CNN
 F 2 "Resistors_SMD:R_0805" V 9880 2700 30  0001 C CNN
@@
 $EndComp
 $Comp
-L R R16
+L R R17
 U 1 1 528E23CA
 P 9700 3350
-F 0 "R16" V 9780 3350 40  0000 C CNN
+F 0 "R17" V 9780 3350 40  0000 C CNN
 F 1 "12k" V 9707 3351 40  0000 C CNN
 F 2 "Resistors_SMD:R_0805" V 9630 3350 30  0001 C CNN
@@
 $EndComp
 $Comp
-L GND #PWR042
+L GND #PWR043
 U 1 1 528E24E6
 P 9700 3700
-F 0 "#PWR042" H 9700 3700 30  0001 C CNN
+F 0 "#PWR043" H 9700 3700 30  0001 C CNN
 F 1 "GND" H 9700 3630 30  0001 C CNN
 F 2 "" H 9700 3700 60  0000 C CNN
@@
 $EndComp
 $Comp
-L GND #PWR043
+L GND #PWR044
 U 1 1 528E25C2
 P 10200 3150
-F 0 "#PWR043" H 10200 3150 30  0001 C CNN
+F 0 "#PWR044" H 10200 3150 30  0001 C CNN
 F 1 "GND" H 10200 3080 30  0001 C CNN
 F 2 "" H 10200 3150 60  0000 C CNN
@@
 $EndComp
 $Comp
-L GND #PWR044
+L GND #PWR045
 U 1 1 528E27BA
 P 7550 3550
-F 0 "#PWR044" H 7550 3550 30  0001 C CNN
+F 0 "#PWR045" H 7550 3550 30  0001 C CNN
 F 1 "GND" H 7550 3480 30  0001 C CNN
 F 2 "" H 7550 3550 60  0000 C CNN
@@
 $EndComp
 $Comp
-L R R11
+L R R12
 U 1 1 528FCEBC
 P 1550 5950
-F 0 "R11" V 1630 5950 40  0000 C CNN
+F 0 "R12" V 1630 5950 40  0000 C CNN
 F 1 "470R" V 1557 5951 40  0000 C CNN
 F 2 "Resistors_SMD:R_0805" V 1480 5950 30  0001 C CNN
@@
 $EndComp
 $Comp
-L GND #PWR045
+L GND #PWR046
 U 1 1 528FD63C
 P 1550 7000
-F 0 "#PWR045" H 1550 7000 30  0001 C CNN
+F 0 "#PWR046" H 1550 7000 30  0001 C CNN
 F 1 "GND" H 1550 6930 30  0001 C CNN
 F 2 "" H 1550 7000 60  0000 C CNN
@@
 P 1550 6600
 F 0 "BT1" H 1550 6800 50  0000 C CNN
-F 1 "ML2016" H 1550 6410 50  0000 C CNN
+F 1 "3V LiMnO2" H 1550 6410 50  0000 C CNN
 F 2 "jakub:ML2016" H 1550 6600 60  0001 C CNN
 F 3 "ML2016.pdf" H 1550 6600 60  0001 C CNN
-F 4 "ML 2016 T6" H 1550 6600 60  0001 C CNN "Part Number"
+F 4 "ML2016 T6" H 1550 6600 60  0001 C CNN "Part Number"
 F 5 "Maxell" H 1550 6600 60  0001 C CNN "Manufacturer"
 F 6 "3031962" H 1550 6600 60  0001 C CNN "Order Code"
@@
 NoConn ~ 1950 5400
 $Comp
-L +3V3 #PWR046
+L +3V3 #PWR047
 U 1 1 54E0A2C9
 P 950 5300
-F 0 "#PWR046" H 950 5150 60  0001 C CNN
+F 0 "#PWR047" H 950 5150 60  0001 C CNN
 F 1 "+3V3" H 950 5440 60  0000 C CNN
 F 2 "" H 950 5300 60  0000 C CNN
@@
 $EndComp
 $Comp
-L +BATT #PWR047
+L +BATT #PWR048
 U 1 1 54E0A3B4
 P 2150 5400
-F 0 "#PWR047" H 2150 5250 60  0001 C CNN
+F 0 "#PWR048" H 2150 5250 60  0001 C CNN
 F 1 "+BATT" H 2150 5540 60  0000 C CNN
 F 2 "" H 2150 5400 60  0000 C CNN
@@
 $EndComp
 $Comp
-L +12V #PWR048
+L +12V #PWR049
 U 1 1 54E0AC5D
 P 1550 2100
-F 0 "#PWR048" H 1550 1950 60  0001 C CNN
+F 0 "#PWR049" H 1550 1950 60  0001 C CNN
 F 1 "+12V" H 1550 2240 60  0000 C CNN
 F 2 "" H 1550 2100 60  0000 C CNN
@@
 $EndComp
 $Comp
-L +12V #PWR049
+L +12V #PWR050
 U 1 1 54E0ACAD
 P 950 2100
-F 0 "#PWR049" H 950 1950 60  0001 C CNN
+F 0 "#PWR050" H 950 1950 60  0001 C CNN
 F 1 "+12V" H 950 2240 60  0000 C CNN
 F 2 "" H 950 2100 60  0000 C CNN
@@
 $EndComp
 $Comp
-L +12V #PWR050
+L +12V #PWR051
 U 1 1 54E0B16A
 P 6100 2100
-F 0 "#PWR050" H 6100 1950 60  0001 C CNN
+F 0 "#PWR051" H 6100 1950 60  0001 C CNN
 F 1 "+12V" H 6100 2240 60  0000 C CNN
 F 2 "" H 6100 2100 60  0000 C CNN
@@
 $EndComp
 $Comp
-L +2V5 #PWR051
+L +2V5 #PWR052
 U 1 1 54E0B844
 P 10200 2300
-F 0 "#PWR051" H 10200 2150 60  0001 C CNN
+F 0 "#PWR052" H 10200 2150 60  0001 C CNN
 F 1 "+2V5" H 10200 2440 60  0000 C CNN
 F 2 "" H 10200 2300 60  0000 C CNN
@@
 $EndComp
 $Comp
-L +3V3 #PWR052
+L +3V3 #PWR053
 U 1 1 54E0DE71
 P 6000 5600
-F 0 "#PWR052" H 6000 5450 60  0001 C CNN
+F 0 "#PWR053" H 6000 5450 60  0001 C CNN
 F 1 "+3V3" H 6000 5740 60  0000 C CNN
 F 2 "" H 6000 5600 60  0000 C CNN
@@
 $EndComp
 $Comp
-L +5VP #PWR053
+L +5VP #PWR054
 U 1 1 54E0DEC7
 P 5000 5600
-F 0 "#PWR053" H 5000 5450 60  0001 C CNN
+F 0 "#PWR054" H 5000 5450 60  0001 C CNN
 F 1 "+5VP" H 5000 5740 60  0000 C CNN
 F 2 "" H 5000 5600 60  0000 C CNN
@@
 $EndComp
 $Comp
-L +5VP #PWR054
+L +5VP #PWR055
 U 1 1 54E0E2E9
 P 4950 2250
-F 0 "#PWR054" H 4950 2100 60  0001 C CNN
+F 0 "#PWR055" H 4950 2100 60  0001 C CNN
 F 1 "+5VP" H 4950 2390 60  0000 C CNN
 F 2 "" H 4950 2250 60  0000 C CNN
@@
 $EndComp
 $Comp
-L GND #PWR055
+L GND #PWR056
 U 1 1 54E0E8FB
 P 5500 6300
-F 0 "#PWR055" H 5500 6050 60  0001 C CNN
+F 0 "#PWR056" H 5500 6050 60  0001 C CNN
 F 1 "GND" H 5500 6150 60  0000 C CNN
 F 2 "" H 5500 6300 60  0000 C CNN

Commit message: Fixed 12k resistor, added .gitignore
Parts:
- R17: Alt. Order Code (none) -> 667-ERJ-6ENF1202V; Alt. Supplier (none) -> Mouser; Note (none) -> 12kΩ/1% 0805 resistor; Order Code 9332502 -> 2447563; Package (none) -> 0805; Part Number MC01W0805112K -> MCWR08X1202FTL; Supplier (none) -> Farnell
Changed lines of the file:
@@
 F 2 "Resistors_SMD:R_0805" V 9630 3350 30  0001 C CNN
 F 3 "" H 9700 3350 30  0000 C CNN
-F 4 "MC01W0805112K" V 9700 3350 60  0001 C CNN "Part Number"
+F 4 "MCWR08X1202FTL" V 9700 3350 60  0001 C CNN "Part Number"
 F 5 "Multicomp" V 9700 3350 60  0001 C CNN "Manufacturer"
-F 6 "9332502" V 9700 3350 60  0001 C CNN "Order Code"
+F 6 "0805" H 9700 3350 60  0001 C CNN "Package"
+F 7 "Farnell" H 9700 3350 60  0001 C CNN "Supplier"
+F 8 "2447563" V 9700 3350 60  0001 C CNN "Order Code"
+F 9 "Mouser" H 9700 3350 60  0001 C CNN "Alt. Supplier"
+F 10 "667-ERJ-6ENF1202V" H 9700 3350 60  0001 C CNN "Alt. Order Code"
+F 11 "12kΩ/1% 0805 resistor" H 9700 3350 60  0001 C CNN "Note"
 	1    9700 3350
 	1    0    0    -1

Commit message: Changed BAR43S diode into 1N4148 for minimum leakage current.
Parts:
- removed D3: BAR43S, Housings_SOT-23_SOT-143_TSOT-6:SOT-23, symbol BAR43S
- added D3: 1N4148, Diodes_SMD:SOD-323, symbol D
Connections:
- net +3V3: now also D3.2 (A)
- net +BATT: now also D3.1 (K)
- no-connect marks 4 -> 3
Changed lines of the file:
@@
 $EndComp
-$Comp
-L BAR43S D3
-U 1 1 532A270B
-P 1550 5400
-F 0 "D3" H 1650 5300 40  0000 C CNN
-F 1 "BAR43S" H 1550 5500 40  0000 C CNN
-F 2 "Housings_SOT-23_SOT-143_TSOT-6:SOT-23" H 1550 5400 60  0001 C CNN
-F 3 "" H 1550 5400 60  0000 C CNN
-F 4 "BAR43SFILM" H 1550 5400 60  0001 C CNN "Part Number"
-F 5 "ST Microelectronics" H 1550 5400 60  0001 C CNN "Manufacturer"
-F 6 "9801391" H 1550 5400 60  0001 C CNN "Order Code"
-	1    1550 5400
-	1    0    0    -1
-$EndComp
-NoConn ~ 1950 5400
 $Comp
 L +3V3 #PWR047
 U 1 1 54E0A2C9
-P 950 5300
-F 0 "#PWR047" H 950 5150 60  0001 C CNN
-F 1 "+3V3" H 950 5440 60  0000 C CNN
-F 2 "" H 950 5300 60  0000 C CNN
-F 3 "" H 950 5300 60  0000 C CNN
-	1    950  5300
+P 950 5400
+F 0 "#PWR047" H 950 5250 60  0001 C CNN
+F 1 "+3V3" H 950 5540 60  0000 C CNN
+F 2 "" H 950 5400 60  0000 C CNN
+F 3 "" H 950 5400 60  0000 C CNN
+	1    950  5400
 	1    0    0    -1
 $EndComp
@@
 	1550 6300 1550 6100
 Wire Wire Line
-	1550 5600 1550 5800
-Wire Wire Line
-	1150 5400 950  5400
-Wire Wire Line
-	950  5400 950  5300
-Wire Wire Line
-	1550 5650 2150 5650
+	950  5650 950  5400
+Wire Wire Line
+	1400 5650 2150 5650
 Wire Wire Line
 	2150 5650 2150 5400
@@
 Text Label 1650 2950 2    60   ~ 0
 SYNC
+$Comp
+L D D3
+U 1 1 56CB3BCC
+P 1250 5650
+F 0 "D3" H 1250 5750 50  0000 C CNN
+F 1 "1N4148" H 1250 5550 50  0000 C CNN
+F 2 "Diodes_SMD:SOD-323" H 1250 5650 50  0001 C CNN
+F 3 "" H 1250 5650 50  0000 C CNN
+F 4 "1N4148WS" H 1250 5650 60  0001 C CNN "Part Number"
+F 5 "Multicomp" H 1250 5650 60  0001 C CNN "Manufacturer"
+F 6 "SOD-323" H 1250 5650 60  0001 C CNN "Package"
+F 7 "Farnell" H 1250 5650 60  0001 C CNN "Supplier"
+F 8 "1466524" H 1250 5650 60  0001 C CNN "Order Code"
+F 9 "Mouser" H 1250 5650 60  0001 C CNN "Alt. Supplier"
+F 10 "512-1N4148WS" H 1250 5650 60  0001 C CNN "Alt. Order Code"
+F 11 "Small signal SOD-323 diode" H 1250 5650 60  0001 C CNN "Note"
+	1    1250 5650
+	-1   0    0    1
+$EndComp
+Wire Wire Line
+	1100 5650 950  5650
+Wire Wire Line
+	1550 5800 1550 5650
 $EndSCHEMATC

Commit message: Added detailed part descriptions
Parts:
- removed C22: 22u/25V, Capacitors_SMD:C_1210, symbol C
- removed C23: 1u, Capacitors_SMD:C_0805, symbol C
- removed C35: 47u/6.3V, Capacitors_SMD:C_1210, symbol C
- added C14: 22u/25V, Capacitors_SMD:C_1210, symbol C
- added C15: 1u/50V, Capacitors_SMD:C_0805, symbol C
- added C19: 47u/16V, Capacitors_SMD:C_1210, symbol C
- BT1: value 3V LiMnO2 -> 3V LiMnO₂; Alt. Order Code (none) -> N/A; Alt. Supplier (none) -> N/A; Note (none) -> Horizontal lithium manganese dioxide rechargeable battery; Package (none) -> ø20mm; Supplier (none) -> Farnell
- C11: value 1u -> 1u/50V; Alt. Order Code (none) -> 81-GRM219R61H105KA3D; Alt. Supplier (none) -> Mouser; Note (none) -> 1μF/50V X5R 0805 ceramic capacitor; Package (none) -> 0805; Supplier (none) -> Farnell
- C12, C28: Alt. Order Code (none) -> 710-885012207098; Alt. Supplier (none) -> Mouser; Note (none) -> 100nF/50V X7R 0805 ceramic capacitor; Package (none) -> 0805; Supplier (none) -> Farnell
- C12, C13: Alt. Order Code (none) -> 74-T55A106M010C0200; Alt. Supplier (none) -> Mouser; Note (none) -> 10μF/10V/0.2Ω ESR case A tantalum capacitor; Package (none) -> case A; Supplier (none) -> Farnell
- C15: value 47u/6.3V -> 47u/16V; Alt. Order Code (none) -> 81-GRM32ER61C476ME15; Alt. Supplier (none) -> Mouser; Note (none) -> 47μF/16V X5R 1210 ceramic capacitor; Order Code 9527788 -> 1735538; Package (none) -> 1210; Part Number GRM32ER60J476ME20L -> GRM32ER61C476ME15L; Supplier (none) -> Farnell
- C17: value 47u/6.3V -> 47u/16V; Alt. Order Code (none) -> 81-GRM32ER61C476ME15; Alt. Supplier (none) -> Mouser; Note (none) -> 47μF/16V X5R 1210 ceramic capacitor; Package (none) -> 1210; Part Number GRM32ER60J476ME20L -> GRM32ER61C476ME15L; Supplier (none) -> Farnell
- C24: Alt. Order Code (none) -> 581-08055C822K; Alt. Supplier (none) -> Mouser; Note (none) -> 8.2nF/50V X7R 0805 ceramic capacitor; Package (none) -> 0805; Part Number MCCA000367 -> MC0805B822K500CT; Supplier (none) -> Farnell
- C31: Alt. Order Code (none) -> 603-CC805CRNPO9BN4R7; Alt. Supplier (none) -> Mouser; Note (none) -> 4.7pF/200V C0G(NP0) 0805 ceramic capacitor; Order Code 1856076 -> 1855762; Package (none) -> 0805; Part Number MCMT18N4R7C100CT -> MC0805N4R7C201CT; Supplier (none) -> Farnell
- C5: Alt. Order Code (none) -> 81-GRM32ER61E226ME5L; Alt. Supplier (none) -> Mouser; Note (none) -> 22μF/25V X5R 1210 ceramic capacitor; Order Code 1828821 -> 1735539; Package (none) -> 1210; Part Number GRM32ER61E226KE15L -> GRM32ER61E226ME15L; Supplier (none) -> Farnell
- C7: Alt. Order Code (none) -> 710-885012207059; Alt. Supplier (none) -> Mouser; Note (none) -> 680pF/50V X7R 0805 ceramic capacitor; Order Code 1856232 -> 1759222; Package (none) -> 0805; Part Number MCCA001064 -> MC0805B681K500CT; Supplier (none) -> Farnell
- C9: Alt. Order Code (none) -> 77-VJ0805A1R5BXAPBC; Alt. Supplier (none) -> Mouser; Note (none) -> 1.5pF/50V C0G(NP0) 0805 ceramic capacitor; Package (none) -> 0805; Part Number MCCA000309 -> MC0805N1R5C500CT; Supplier (none) -> Farnell
- L1: Alt. Order Code (none) -> 70-IHLP4040DZER3R3M0; Alt. Supplier (none) -> Mouser; Note (none) -> 3.3μH 10A low profile high current IHLP inductor; Package (none) -> 10.3mm×10.3mm; Supplier (none) -> Farnell
- L5: Alt. Order Code (none) -> 70-IHLP3232DZER2R2M1; Alt. Supplier (none) -> Mouser; Note (none) -> 2.2μH 14.5A low profile high current IHLP inductor; Package (none) -> 8.2mm×8.2mm; Supplier (none) -> Farnell
- Q4: Alt. Order Code (none) -> 942-IRF8721PBF; Alt. Supplier (none) -> Mouser; Note (none) -> N-channel SOIC-8 MOSFET; Package (none) -> SOIC-8; Supplier (none) -> Farnell
- R11, R13: Alt. Order Code (none) -> 71-CRCW0805-82K-E3; Alt. Supplier (none) -> Mouser; Note (none) -> 82kΩ/1% 0805 resistor; Package (none) -> 0805; Supplier (none) -> Farnell
- R12: Alt. Order Code (none) -> 667-ERJ-6ENF4700V; Alt. Supplier (none) -> Mouser; Note (none) -> 470Ω/1% 0805 resistor; Package (none) -> 0805; Supplier (none) -> Farnell
- R14: Alt. Order Code (none) -> 71-CRCW0805-22K-E3; Alt. Supplier (none) -> Mouser; Note (none) -> 22kΩ/1% 0805 resistor; Package (none) -> 0805; Supplier (none) -> Farnell
- R15: Alt. Order Code (none) -> 667-ERJ-6GEYJ302V; Alt. Supplier (none) -> Mouser; Note (none) -> 3kΩ/1% 0805 resistor; Package (none) -> 0805; Supplier (none) -> Farnell
- R16: Alt. Order Code (none) -> 71-CRCW0805-10K-E3; Alt. Supplier (none) -> Mouser; Note (none) -> 10kΩ/1% 0805 resistor; Package (none) -> 0805; Supplier (none) -> Farnell
- R18: Alt. Order Code (none) -> 667-ERJ-6ENF3302V; Alt. Supplier (none) -> Mouser; Note (none) -> 33kΩ/1% 0805 resistor; Package (none) -> 0805; Supplier (none) -> Farnell
- U1: Alt. Order Code (none) -> 621-AP1117E33G-13; Alt. Supplier (none) -> Mouser; Note (none) -> 3.3V linear voltage regulator; Package (none) -> SOT-223; Supplier (none) -> Farnell
- U2: Alt. Order Code (none) -> 584-ADP2381AREZ-R7; Alt. Supplier (none) -> Mouser; Note (none) -> 20V 6A synchronous step-down regulator with low-side driver; Package (none) -> PowerPAD TSSOP-16; Supplier (none) -> Farnell
- U3: Alt. Order Code (none) -> 595-TPS54428DDA; Alt. Supplier (none) -> Mouser; Note (none) -> 4.5-18V input 4A synchronous step-down converter with eco-m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; Package (none) -> PowerPAD SOIC-8; Supplier (none) -> Farnell
Connections:
- net +12V: now also C14.1
- net +2V5: now also C19.1
- net GND: now also C14.2, C15.2, C19.2
- net VREG2.8: now also C15.1
