File: MicroFLiC_power_supply.kicad_pcb (KiCad board)
At the start: 2 copper layers, 49.8 x 49.8 mm, 65 parts, among them P1 DC jack, P2 6-way Micro-MaTch, P3 1x14 socket strip, P4 2x2 socket strip, P6 1x3 header strip, Q1 SI2369, Q2 TSM2314, Q3 SI2369, Q4 IRF8721, SW1 Tactile switch R/A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

Commit message: Changed SOD-323 package for easier soldering, fixed Avago->Broadcom LED manufacturer
Parts:
- D1, D2, D3: footprint Diodes_SMD:SOD-323 -> jakub:SOD-323
Changed lines of the file:
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@@
     (pad_to_mask_clearance 0)
     (aux_axis_origin 100.076 149.86)
-    (visible_elements FFFFFF7F)
+    (visible_elements FFFEFF7F)
     (pcbplotparams
       (layerselection 0x010f0_80000001)
@@
     )
   )
-  (module Diodes_SMD:SOD-323 (layer F.Cu)
+  (module Resistors_SMD:R_0805 (layer F.Cu)
+    (at 123.19 118.044 270)
+    (descr "Resistor SMD 0805, reflow soldering, Vishay (see dcrcw.pdf)")
+    (tags "resistor 0805")
+    (attr smd)
+    (fp_text reference R10 (at -0.188 1.524 270) (layer F.SilkS)
+      (effects (font (size 0.8 0.8) (thickness 0.12)))
+    )
+    (fp_text value 10k (at 0 2.1 270) (layer F.Fab) hide
+      (effects (font (size 1 1) (thickness 0.15)))
+    )
+    (fp_line (start -1.6 -1) (end 1.6 -1) (layer F.CrtYd) (width 0.05))
+    (fp_line (start -1.6 1) (end 1.6 1) (layer F.CrtYd) (width 0.05))
+    (fp_line (start -1.6 -1) (end -1.6 1) (layer F.CrtYd) (width 0.05))
+    (fp_line (start 1.6 -1) (end 1.6 1) (layer F.CrtYd) (width 0.05))
+    (fp_line (start 0.6 0.875) (end -0.6 0.875) (layer F.SilkS) (width 0.15))
+    (fp_line (start -0.6 -0.875) (end 0.6 -0.875) (layer F.SilkS) (width 0.15))
+    (pad 1 smd rect (at -0.95 0 270) (size 0.7 1.3) (layers F.Cu F.Paste F.Mask)
+      (net 6 +12V))
+    (pad 2 smd rect (at 0.95 0 270) (size 0.7 1.3) (layers F.Cu F.Paste F.Mask)
+      (net 2 GND))
+    (model Resistors_SMD.3dshapes/R_0805.wrl
+      (at (xyz 0 0 0))
+      (scale (xyz 1 1 1))
+      (rotate (xyz 0 0 0))
+    )
+  )
+  (module jakub:SOD-323 (layer F.Cu)
     (at 132.588 109.474 270)
     (descr SOD-323)
     (tags SOD-323)
     (attr smd)
-    (fp_text reference D1 (at -0.762 1.778 360) (layer F.SilkS)
-      (effects (font (size 0.8 0.8) (thickness 0.12)))
-    )
-    (fp_text value 1N4148 (at 0.1 1.9 270) (layer F.Fab) hide
+    (fp_text reference D1 (at -2.032 0 360) (layer F.SilkS)
+      (effects (font (size 0.7 0.7) (thickness 0.11)))
+    )
+    (fp_text value 1N4148 (at 0.1 1.9 270) (layer F.Fab)
       (effects (font (size 1 1) (thickness 0.15)))
     )
@@
     (fp_line (start -1.3 0.8) (end 1.1 0.8) (layer F.SilkS) (width 0.15))
     (fp_line (start -1.3 -0.8) (end 1.1 -0.8) (layer F.SilkS) (width 0.15))
-    (pad 1 smd rect (at -1.055 0 270) (size 0.59 0.45) (layers F.Cu F.Paste F.Mask)
+    (pad 1 smd rect (at -1.055 0 270) (size 0.9 0.9) (layers F.Cu F.Paste F.Mask)
       (net 4 /electronicSwitch/PUSHBUTTON))
-    (pad 2 smd rect (at 1.055 0 270) (size 0.59 0.45) (layers F.Cu F.Paste F.Mask)
+    (pad 2 smd rect (at 1.055 0 270) (size 0.9 0.9) (layers F.Cu F.Paste F.Mask)
       (net 12 /electronicSwitch/MCU_OFF))
     (model jakub.3dshapes/diodes/sod323.wrl
@@
     )
   )
-  (module Diodes_SMD:SOD-323 (layer F.Cu)
+  (module jakub:SOD-323 (layer F.Cu)
     (at 123.444 115.316)
     (descr SOD-323)
@@
     (attr smd)
     (fp_text reference D2 (at 2.286 0.508) (layer F.SilkS)
-      (effects (font (size 0.8 0.8) (thickness 0.12)))
-    )
-    (fp_text value 1N4148 (at 0.1 1.9) (layer F.Fab) hide
+      (effects (font (size 0.7 0.7) (thickness 0.11)))
+    )
+    (fp_text value 1N4148 (at 0.1 1.9) (layer F.Fab)
       (effects (font (size 1 1) (thickness 0.15)))
     )
@@
     (fp_line (start -1.3 0.8) (end 1.1 0.8) (layer F.SilkS) (width 0.15))
     (fp_line (start -1.3 -0.8) (end 1.1 -0.8) (layer F.SilkS) (width 0.15))
-    (pad 1 smd rect (at -1.055 0) (size 0.59 0.45) (layers F.Cu F.Paste F.Mask)
+    (pad 1 smd rect (at -1.055 0) (size 0.9 0.9) (layers F.Cu F.Paste F.Mask)
       (net 7 /electronicSwitch/CURLIM))
-    (pad 2 smd rect (at 1.055 0) (size 0.59 0.45) (layers F.Cu F.Paste F.Mask)
+    (pad 2 smd rect (at 1.055 0) (size 0.9 0.9) (layers F.Cu F.Paste F.Mask)
       (net 3 "Net-(C1-Pad1)"))
     (model jakub.3dshapes/diodes/sod323.wrl
@@
     )
   )
-  (module Resistors_SMD:R_0805 (layer F.Cu)
-    (at 123.19 118.044 270)
-    (descr "Resistor SMD 0805, reflow soldering, Vishay (see dcrcw.pdf)")
-    (tags "resistor 0805")
-    (attr smd)
-    (fp_text reference R10 (at -0.188 1.524 270) (layer F.SilkS)
-      (effects (font (size 0.8 0.8) (thickness 0.12)))
-    )
-    (fp_text value 10k (at 0 2.1 270) (layer F.Fab) hide
-      (effects (font (size 1 1) (thickness 0.15)))
-    )
-    (fp_line (start -1.6 -1) (end 1.6 -1) (layer F.CrtYd) (width 0.05))
-    (fp_line (start -1.6 1) (end 1.6 1) (layer F.CrtYd) (width 0.05))
-    (fp_line (start -1.6 -1) (end -1.6 1) (layer F.CrtYd) (width 0.05))
-    (fp_line (start 1.6 -1) (end 1.6 1) (layer F.CrtYd) (width 0.05))
-    (fp_line (start 0.6 0.875) (end -0.6 0.875) (layer F.SilkS) (width 0.15))
-    (fp_line (start -0.6 -0.875) (end 0.6 -0.875) (layer F.SilkS) (width 0.15))
-    (pad 1 smd rect (at -0.95 0 270) (size 0.7 1.3) (layers F.Cu F.Paste F.Mask)
-      (net 6 +12V))
-    (pad 2 smd rect (at 0.95 0 270) (size 0.7 1.3) (layers F.Cu F.Paste F.Mask)
-      (net 2 GND))
-    (model Resistors_SMD.3dshapes/R_0805.wrl
-      (at (xyz 0 0 0))
-      (scale (xyz 1 1 1))
-      (rotate (xyz 0 0 0))
-    )
-  )
-  (module Diodes_SMD:SOD-323 (layer B.Cu)
+  (module jakub:SOD-323 (layer B.Cu)
     (at 111.76 142.748 180)
     (descr SOD-323)
     (tags SOD-323)
     (attr smd)
-    (fp_text reference D3 (at 2.286 0 180) (layer B.SilkS)
-      (effects (font (size 0.8 0.8) (thickness 0.12)) (justify mirror))
+    (fp_text reference D3 (at 0 1.27 180) (layer B.SilkS)
+      (effects (font (size 0.7 0.7) (thickness 0.11)) (justify mirror))
     )
     (fp_text value 1N4148 (at 0.1 -1.9 180) (layer B.Fab)
@@
     (fp_line (start -1.3 -0.8) (end 1.1 -0.8) (layer B.SilkS) (width 0.15))
     (fp_line (start -1.3 0.8) (end 1.1 0.8) (layer B.SilkS) (width 0.15))
-    (pad 1 smd rect (at -1.055 0 180) (size 0.59 0.45) (layers B.Cu B.Paste B.Mask)
+    (pad 1 smd rect (at -1.055 0 180) (size 0.9 0.9) (layers B.Cu B.Paste B.Mask)
       (net 15 +BATT))
-    (pad 2 smd rect (at 1.055 0 180) (size 0.59 0.45) (layers B.Cu B.Paste B.Mask)
+    (pad 2 smd rect (at 1.055 0 180) (size 0.9 0.9) (layers B.Cu B.Paste B.Mask)
       (net 10 +3V3))
+    (model jakub.3dshapes/diodes/sod323.wrl
+      (at (xyz 0 0 0))
+      (scale (xyz 1 1 1))
+      (rotate (xyz 0 0 180))
+    )
   )
   (gr_line (start 131.572 119.888) (end 121.92 119.888) (layer F.SilkS) (width 0.2))
