File: MicroFLiC_power_supply.sch (KiCad schematic (older format))
At the start: 17 parts, among them P1 DC jack, P2 6-way Micro-MaTch, P3 1x14 socket strip, P4 2x2 socket strip, SW1 Tactile switch R/A

Commit message: Changed SOD-323 package for easier soldering, fixed Avago->Broadcom LED manufacturer
Parts:
- D4: Manufacturer Avago -> Croadcom
- D5, D6, D7: Manufacturer Avago -> Broadcom
Changed lines of the file:
@@
 F 3 "" H 9050 2500 60  0000 C CNN
 F 4 "HSMY-C150" H 9050 2500 60  0001 C CNN "Part Number"
-F 5 "Avago" H 9050 2500 60  0001 C CNN "Manufacturer"
+F 5 "Croadcom" H 9050 2500 60  0001 C CNN "Manufacturer"
 F 6 "1206" H 9050 2500 60  0001 C CNN "Package"
 F 7 "Farnell" H 9050 2500 60  0001 C CNN "Supplier"
@@
 F 3 "" H 9350 2500 60  0000 C CNN
 F 4 "HSMY-C150" H 9350 2500 60  0001 C CNN "Part Number"
-F 5 "Avago" H 9350 2500 60  0001 C CNN "Manufacturer"
+F 5 "Broadcom" H 9350 2500 60  0001 C CNN "Manufacturer"
 F 6 "1206" H 9350 2500 60  0001 C CNN "Package"
 F 7 "Farnell" H 9350 2500 60  0001 C CNN "Supplier"
@@
 F 3 "" H 9650 2500 60  0000 C CNN
 F 4 "HSMY-C150" H 9650 2500 60  0001 C CNN "Part Number"
-F 5 "Avago" H 9650 2500 60  0001 C CNN "Manufacturer"
+F 5 "Broadcom" H 9650 2500 60  0001 C CNN "Manufacturer"
 F 6 "1206" H 9650 2500 60  0001 C CNN "Package"
 F 7 "Farnell" H 9650 2500 60  0001 C CNN "Supplier"
@@
 F 3 "" H 9950 2500 60  0000 C CNN
 F 4 "HSMY-C150" H 9950 2500 60  0001 C CNN "Part Number"
-F 5 "Avago" H 9950 2500 60  0001 C CNN "Manufacturer"
+F 5 "Broadcom" H 9950 2500 60  0001 C CNN "Manufacturer"
 F 6 "1206" H 9950 2500 60  0001 C CNN "Package"
 F 7 "Farnell" H 9950 2500 60  0001 C CNN "Supplier"
