File: PowerSupply.sch (KiCad schematic (older format))
At the start: 31 parts, among them Q4 IRF8721, U1 AP1117E33, U2 ADP2381, U3 TPS54428

Commit message: Changed SOD-323 package for easier soldering, fixed Avago->Broadcom LED manufacturer
Parts:
- D3: footprint Diodes_SMD:SOD-323 -> jakub:SOD-323
Changed lines of the file:
@@
 F 0 "D3" H 1250 5750 50  0000 C CNN
 F 1 "1N4148" H 1250 5550 50  0000 C CNN
-F 2 "Diodes_SMD:SOD-323" H 1250 5650 50  0001 C CNN
+F 2 "jakub:SOD-323" H 1250 5650 50  0001 C CNN
 F 3 "" H 1250 5650 50  0000 C CNN
 F 4 "1N4148WS" H 1250 5650 60  0001 C CNN "Part Number"
