File: electronicSwitch.sch (KiCad schematic (older format))
At the start: 17 parts, among them P6 1x3 header strip, Q1 SI2369, Q2 TSM2314, Q3 SI2369

Commit message: Changed SOD-323 package for easier soldering, fixed Avago->Broadcom LED manufacturer
Parts:
- D1, D2: footprint Diodes_SMD:SOD-323 -> jakub:SOD-323
Changed lines of the file:
@@
 F 0 "D2" H 6800 2950 40  0000 C CNN
 F 1 "1N4148" H 6800 3150 40  0000 C CNN
-F 2 "Diodes_SMD:SOD-323" H 6800 3050 50  0001 C CNN
+F 2 "jakub:SOD-323" H 6800 3050 50  0001 C CNN
 F 3 "" H 6800 3050 50  0000 C CNN
 F 4 "1N4148WS" H 6800 3050 60  0001 C CNN "Part Number"
@@
 F 0 "D1" V 4450 3550 40  0000 L CNN
 F 1 "1N4148" V 4550 3550 40  0000 L CNN
-F 2 "Diodes_SMD:SOD-323" H 4500 3450 50  0001 C CNN
+F 2 "jakub:SOD-323" H 4500 3450 50  0001 C CNN
 F 3 "" H 4500 3450 50  0000 C CNN
 F 4 "1N4148WS" H 4500 3450 60  0001 C CNN "Part Number"
